File: flying thing that crashes/flying thing that crashes.kicad_pcb (KiCad board)
At the start: 2 copper layers, 83 parts, among them J1 RMotor, J2 LMotor, J3 J3, J4 J4, M1 Motor_Servo, M2 Motor_Servo, M3 Motor_Servo, M4 Motor_Servo, M5 Motor_Servo, M6 Motor_Servo, M7 Motor_Servo, M8 Motor_Servo, U1 PCA9685PW, U2 Ai-Thinker-Ra-02, U3 Ai-Thinker-Ra-02, U4 AMS1117-3.3, U5 MPU-9250, U6 TPS63070RNMR

Commit message: update(almost done)
Parts:
- moved C1 65.9 mm to (85.0, 46.3), turned to 90 degrees
- moved U1 57.4 mm to (78.5, 46.0), turned to 90 degrees
- moved R1 49.1 mm to (72.0, 46.0), turned to 90 degrees
- moved J5 40.3 mm to (70.5, 36.5)
- moved J6 40.3 mm to (70.5, 32.5)
- moved C18 23.5 mm to (21.9, 82.5)
- moved C19 23.5 mm to (28.4, 82.5)
- moved C16 23.5 mm to (48.0, 82.0)
- moved C17 23.5 mm to (43.0, 82.0)
- moved C2 6.05 mm to (84.5, 60.3)
- moved C3 6.05 mm to (88.0, 60.5)
- moved C4 6.05 mm to (108.5, 60.3)
- moved C5 6.05 mm to (103.5, 60.5)
- moved U4 6.05 mm to (95.5, 60.5)
- moved R31 5.78 mm to (98.0, 45.3), turned to 180 degrees
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Connections:
- C16 pad 1: Net-(U2-VDD) -> 3V3
- C16 pad 2: 3V3 -> GND
- C17 pad 1: 3V3 -> GND
- C17 pad 2: Net-(U2-VDD) -> 3V3
- C18 pad 1: 3V3 -> GND
- C18 pad 2: Net-(U3-VDD) -> 3V3
- C19 pad 1: Net-(U3-VDD) -> 3V3
- C19 pad 2: 3V3 -> GND
- U2 pad 3: Net-(U2-VDD) -> 3V3
- U3 pad 3: Net-(U3-VDD) -> 3V3
Routing:
- net D13: track 3.85 -> 155.4 mm, vias 0 -> 6
- net GND: track 107.2 -> 209.8 mm, vias 0 -> 6
- net A3: track 0.00 -> 91.5 mm, vias 0 -> 3
- net A2: track 0.00 -> 83.2 mm, vias 0 -> 6
- net PWM 7: track 0.00 -> 80.6 mm, vias 0 -> 3
- net A1: track 0.00 -> 80.3 mm, vias 0 -> 6
- net PWM 9: track 0.00 -> 77.2 mm, vias 0 -> 3
- net A0: track 0.00 -> 75.7 mm, vias 0 -> 2
- net D12: track 3.85 -> 76.8 mm, vias 0 -> 7
- net PWM 8: track 0.00 -> 67.7 mm, vias 0 -> 3
- net D11: track 3.85 -> 67.7 mm, vias 0 -> 4
- net D4: track 3.85 -> 59.3 mm, vias 0 -> 2
- net Net-(JP4-B): track 0.00 -> 46.0 mm, vias 0 -> 4
- net 5V: track 18.6 -> 64.4 mm, vias 0 -> 5
- net A4: track 6.54 -> 50.5 mm, vias 0 -> 5
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
Commit message: final draft
Parts:
- moved C4 24.2 mm to (88.7, 74.2), turned to 180 degrees
- moved C5 17.3 mm to (88.5, 69.2), turned to 180 degrees
- moved C2 10.9 mm to (88.7, 50.2), turned to 180 degrees
- moved U4 7.03 mm to (88.5, 61.2), turned to 180 degrees
- moved C3 6.87 mm to (88.5, 53.7), turned to 180 degrees
Routing:
- net 3V3: track 69.6 -> 202.3 mm, vias 2 -> 9
- net A7: track 4.05 -> 121.2 mm, vias 0 -> 2
- net A5: track 31.3 -> 134.6 mm, vias 3 -> 8
- net A4: track 50.5 -> 153.2 mm, vias 5 -> 12
- net A6: track 4.05 -> 100.6 mm, vias 0 -> 4
- net 5V: track 64.4 -> 147.9 mm, vias 5 -> 9
- net GND: track 209.8 -> 279.1 mm, vias 6 -> 13
- net Net-(JP3-B): track 6.71 -> 71.5 mm, vias 2 -> 6
- net Net-(JP5-B): track 19.1 -> 79.4 mm, vias 2 -> 8
- net Net-(JP4-B): track 46.0 -> 97.9 mm, vias 4 -> 5
- net Net-(JP2-B): track 14.7 -> 51.9 mm, vias 0 -> 6
- net Net-(JP1-B): track 22.0 -> 50.4 mm, vias 2 -> 4
- net Net-(JP6-B): track 28.4 -> 50.4 mm, vias 2 -> 4
- net PWM 7: track 80.6 -> 89.9 mm, vias 3 -> 5
- net MVIN: track 39.3 -> 38.0 mm

Commit message: tweeks to final draft(cleenup)
Routing:
- net GND: track 279.1 -> 353.2 mm, vias 13 -> 14
- net D12: track 76.8 -> 121.8 mm, vias 7 -> 10
- net D11: track 67.7 -> 110.3 mm, vias 4 -> 7
- net MVIN: track 38.0 -> 0.00 mm
- net Net-(JP1-B): track 50.4 -> 28.4 mm, vias 4 -> 2
- net Net-(JP4-B): track 97.9 -> 85.1 mm, vias 5 -> 4
- net A5: track 134.6 -> 126.9 mm, vias 8 -> 6
- net AD0: track 9.86 -> 12.6 mm, vias 0 -> 2
- net Net-(U5-REGOUT): track 8.66 -> 9.74 mm
- net PWM 9: track 77.2 -> 76.6 mm

Commit message: controller
Parts:
- moved C6 3.81 mm to (65.7, 64.9)
- moved A1 3.81 mm to (32.0, 56.7)
- moved C1 3.81 mm to (83.5, 49.8)
- moved C10 3.81 mm to (69.7, 66.0)
- moved C11 3.81 mm to (57.7, 59.9)
- moved C12 3.81 mm to (62.2, 61.9)
- moved C13 3.81 mm to (96.0, 40.4)
- moved C14 3.81 mm to (96.0, 35.9)
- moved C15 3.81 mm to (91.5, 40.4)
- moved C16 3.81 mm to (46.5, 85.5)
- moved C17 3.81 mm to (41.5, 85.5)
- moved C18 3.81 mm to (20.4, 86.0)
- moved C19 3.81 mm to (26.9, 86.0)
- moved C2 3.81 mm to (87.2, 53.7)
- moved C3 3.81 mm to (87.0, 57.2)
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